File: hardware/piano_proto/projet_piano_proto_kicad.kicad_pcb (KiCad board)
At the start: 2 copper layers, 104.1 x 81.3 mm, 16 parts, among them J1 Screw_Terminal_01x02, SW1 800USP8P1A1M2RE, SW2 EG1218, SW3 800USP8P1A1M2RE, SW4 800USP8P1A1M2RE, SW5 800USP8P1A1M2RE, SW6 800USP8P1A1M2RE, SW7 800USP8P1A1M2RE, U1 CD74HCT251E, U2 CD74HCT251E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

Commit message: First test passed with main boards and all satellite boards connected
Connections:
- A2 pad 4: GND -> Net-(A2-A0)
Changed lines of the file:
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@@
 		)
 		(property "Footprint" "Module:Arduino_Nano"
-			(at 0 0 0)
+			(at 8.875 -18.375 0)
 			(unlocked yes)
 			(layer "F.Fab")
@@
 		)
 		(property "Datasheet" "https://content.arduino.cc/assets/NANOEveryV3.0_sch.pdf"
-			(at 0 0 0)
+			(at 10.5 -14.65 0)
 			(unlocked yes)
 			(layer "F.Fab")
@@
 		)
 		(property "Description" "Arduino Nano Every"
-			(at 0 0 0)
+			(at 8.175 -9.6 0)
 			(unlocked yes)
 			(layer "F.Fab")
@@
 		)
 		(fp_line
-			(start 3.68 31.62)
-			(end 11.56 31.62)
-			(stroke
-				(width 0.12)
-				(type solid)
-			)
-			(layer "F.SilkS")
-		)
-		(fp_line
-			(start 3.68 42.04)
-			(end 3.68 31.62)
-			(stroke
-				(width 0.12)
-				(type solid)
-			)
-			(layer "F.SilkS")
-		)
-		(fp_line
-			(start 11.56 31.62)
-			(end 11.56 42.04)
-			(stroke
-				(width 0.12)
-				(type solid)
-			)
-			(layer "F.SilkS")
-		)
-		(fp_line
-			(start 11.56 42.04)
-			(end 3.68 42.04)
+			(start 3.5 -4.03)
+			(end 11.38 -4.03)
+			(stroke
+				(width 0.12)
+				(type solid)
+			)
+			(layer "F.SilkS")
+		)
+		(fp_line
+			(start 3.5 6.39)
+			(end 3.5 -4.03)
+			(stroke
+				(width 0.12)
+				(type solid)
+			)
+			(layer "F.SilkS")
+		)
+		(fp_line
+			(start 11.38 -4.03)
+			(end 11.38 6.39)
+			(stroke
+				(width 0.12)
+				(type solid)
+			)
+			(layer "F.SilkS")
+		)
+		(fp_line
+			(start 11.38 6.39)
+			(end 3.5 6.39)
 			(stroke
 				(width 0.12)
@@
 		)
 		(fp_line
-			(start 3.81 31.75)
-			(end 11.43 31.75)
-			(stroke
-				(width 0.1)
-				(type solid)
-			)
-			(layer "F.Fab")
-		)
-		(fp_line
-			(start 3.81 41.91)
-			(end 3.81 31.75)
-			(stroke
-				(width 0.1)
-				(type solid)
-			)
-			(layer "F.Fab")
-		)
-		(fp_line
-			(start 11.43 31.75)
-			(end 11.43 41.91)
-			(stroke
-				(width 0.1)
-				(type solid)
-			)
-			(layer "F.Fab")
-		)
-		(fp_line
-			(start 11.43 41.91)
-			(end 3.81 41.91)
+			(start 3.63 -3.9)
+			(end 11.25 -3.9)
+			(stroke
+				(width 0.1)
+				(type solid)
+			)
+			(layer "F.Fab")
+		)
+		(fp_line
+			(start 3.63 6.26)
+			(end 3.63 -3.9)
+			(stroke
+				(width 0.1)
+				(type solid)
+			)
+			(layer "F.Fab")
+		)
+		(fp_line
+			(start 11.25 -3.9)
+			(end 11.25 6.26)
+			(stroke
+				(width 0.1)
+				(type solid)
+			)
+			(layer "F.Fab")
+		)
+		(fp_line
+			(start 11.25 6.26)
+			(end 3.63 6.26)
 			(stroke
 				(width 0.1)
@@
 		)
 		(fp_text user "USB"
-			(at 7.62 35.56 0)
+			(at 7.44 -0.09 0)
 			(unlocked yes)
 			(layer "F.SilkS")
@@
 			(layers "*.Cu" "*.Mask")
 			(remove_unused_layers no)
-			(net 4 "GND")
-			(pinfunction "GND")
-			(pintype "power_in")
+			(net 50 "Net-(A2-A0)")
+			(pinfunction "A0")
+			(pintype "bidirectional")
 		)
 		(pad "5" thru_hole oval
