File: hardware/piano_proto/projet_piano_proto_kicad.kicad_sch (KiCad schematic)
At the start: 16 parts, among them J1 Screw_Terminal_01x02, SW1 800USP8P1A1M2RE, SW2 EG1218, SW3 800USP8P1A1M2RE, SW4 800USP8P1A1M2RE, SW5 800USP8P1A1M2RE, SW6 800USP8P1A1M2RE, SW7 800USP8P1A1M2RE, U1 CD74HCT251E, U2 CD74HCT251E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

Commit message: First test passed with main boards and all satellite boards connected
Connections:
- net GND: no longer A2.4 (GND)
Changed lines of the file:
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@@
 		(on_board yes)
 		(dnp no)
-		(fields_autoplaced yes)
 		(property "Reference" "A2"
-			(at 290.4841 168.91 0)
+			(at 274.066 112.776 0)
 			(effects
 				(font
@@
 				)
 				(justify left)
+				(hide yes)
 			)
 		)
 		(property "Value" "Arduino_Nano_Every"
-			(at 290.4841 171.45 0)
+			(at 265.43 116.332 0)
 			(effects
 				(font
@@
 		)
 		(property "Footprint" "Module:Arduino_Nano"
-			(at 288.29 143.51 0)
+			(at 288.036 100.838 0)
 			(effects
 				(font
@@
 		)
 		(property "Datasheet" "https://content.arduino.cc/assets/NANOEveryV3.0_sch.pdf"
-			(at 288.29 143.51 0)
+			(at 288.036 105.156 0)
 			(effects
 				(font
@@
 		)
 		(property "Description" "Arduino Nano Every"
-			(at 288.29 143.51 0)
+			(at 287.528 97.028 0)
 			(effects
 				(font
@@
 		(pin "27"
 		)
-		(pin "4"
-		)
 		(pin "5"
