File: hardware/satellite_board_6_keys/satellite_board_6_keys.kicad_sch (KiCad schematic)
At the start: 16 parts, among them J1 Conn_01x02_Socket, J2 Conn_01x06_Socket, J3 Conn_01x06_Socket, J4 Conn_02x12_Odd_Even, J5 Conn_02x12_Odd_Even, U1 CD74HCT251E, U2 CD74HCT251E

Commit message: First test passed with main boards and all satellite boards connected
Parts:
- R1: value 1 KOhm -> 4.7 KOhm
- R2: value 4.7 KOhm -> 20 KOhm
Changed lines of the file:
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@@
 			)
 		)
-		(property "Value" "1 KOhm"
+		(property "Value" "4.7 KOhm"
 			(at 71.12 45.72 0)
 			(effects
@@
 			)
 		)
-		(property "Value" "4.7 KOhm"
+		(property "Value" "20 KOhm"
 			(at 124.46 45.72 0)
 			(effects
